Commit message: remove prefix for urdf module

File: dsr_description/urdf/DSR_body.urdf.xacro (robot description, xacro)
@@ -77,7 +77,7 @@
     </xacro:macro>
     <!-- DSR Macro -->
-    <xacro:macro name="DSR_BODY" params="prefix">
+    <xacro:macro name="DSR_BODY">
         <!-- Link: base_footprint -->
-        <link name="${prefix}_base_footprint">
+        <link name="base_footprint">
             <visual>
                 <origin xyz="0 0 0" rpy="0 0 0" />
@@ -88,11 +88,11 @@
         </link>
         <!-- Joint: base_footprint & base_link -->
-        <joint name="${prefix}_base_footprint_joint" type="fixed">
+        <joint name="base_footprint_joint" type="fixed">
             <origin xyz="0 0 -0.005" rpy="0 0 0" />
-            <parent link="${prefix}_base_footprint"/>
-            <child link="${prefix}_base_link" />
+            <parent link="base_footprint"/>
+            <child link="base_link" />
         </joint>
         <!-- Link: base_link -->
-        <link name="${prefix}_base_link">
+        <link name="base_link">
             <xacro:Box_Inertia  m="${base_link_mass}"
                                 x="${base_link_x}"
@@ -118,5 +118,5 @@
         </link>
         <!-- Link: back motor link -->
-        <link name="${prefix}_back_motor_link">
+        <link name="back_motor_link">
             <xacro:Box_Inertia  m="${motor_mass}"
                                 x="${motor_ixx}"
@@ -140,7 +140,7 @@
         </link>
         <!-- Joint: base_link & back motor -->
-        <joint name="${prefix}_joint_back_motor" type="continuous">
-            <parent link="${prefix}_base_link"/>
-            <child link="${prefix}_back_motor_link"/>
+        <joint name="joint_back_motor" type="continuous">
+            <parent link="base_link"/>
+            <child link="back_motor_link"/>
             <origin xyz="-${wheel_offset_x} ${wheel_offset_y} ${motor_wheel_offset_z}" rpy="0 0 0" />
             <axis xyz="0 0 1" rpy="0 0 0" />
@@ -149,10 +149,10 @@
         </joint>
         <!-- Transmission: back motor -->
-        <transmission name="${prefix}_joint_bmw_trans">
-            <type>transmission_interface/SimpleTransmission</type>
-            <joint name="${prefix}_joint_back_motor">
-                <hardwareInterface>hardware_interface/EffortJointInterface</hardwareInterface>
-            </joint>
-            <actuator name="${prefix}_joint_bmw_motor">
+        <transmission name="joint_bmw_trans">
+            <type>transmission_interface/SimpleTransmission</type>
+            <joint name="joint_back_motor">
+                <hardwareInterface>hardware_interface/EffortJointInterface</hardwareInterface>
+            </joint>
+            <actuator name="joint_bmw_motor">
                 <hardwareInterface>hardware_interface/EffortJointInterface</hardwareInterface>
                 <mechanicalReduction>${motor_wheel_mechanical_reduction}</mechanicalReduction>
@@ -160,5 +160,5 @@
         </transmission>
         <!-- Link: back wheel link -->
-        <link name="${prefix}_back_wheel_link">
+        <link name="back_wheel_link">
             <xacro:Wheel_Inertia    m="${wheel_mass}"
                                     ixx="${wheel_ixx}"
@@ -182,7 +182,7 @@
         </link>
         <!-- Joint: back motor & back wheel link -->
-        <joint name="${prefix}_joint_back_wheel" type="continuous">
-            <parent link="${prefix}_back_motor_link"/>
-            <child link="${prefix}_back_wheel_link"/>
+        <joint name="joint_back_wheel" type="continuous">
+            <parent link="back_motor_link"/>
+            <child link="back_wheel_link"/>
             <origin xyz="0 0 0" rpy="0 0 0" />
             <axis xyz="0 1 0" rpy="0 0 0" />
@@ -191,10 +191,10 @@
         </joint>
         <!-- Transmission: back wheel -->
-        <transmission name="${prefix}_joint_bw_trans">
-            <type>transmission_interface/SimpleTransmission</type>
-            <joint name="${prefix}_joint_back_wheel">
+        <transmission name="joint_bw_trans">
+            <type>transmission_interface/SimpleTransmission</type>
+            <joint name="joint_back_wheel">
                 <hardwareInterface>hardware_interface/VelocityJointInterface</hardwareInterface>
             </joint>
-            <actuator name="${prefix}_joint_bw_motor">
+            <actuator name="joint_bw_motor">
                 <hardwareInterface>hardware_interface/VelocityJointInterface</hardwareInterface>
                 <mechanicalReduction>${wheel_mechanical_reduction}</mechanicalReduction>
@@ -202,5 +202,5 @@
         </transmission>
         <!-- Link: front motor link -->
-        <link name="${prefix}_front_motor_link">
+        <link name="front_motor_link">
             <xacro:Box_Inertia  m="${motor_mass}"
                                 x="${motor_ixx}"
@@ -224,7 +224,7 @@
         </link>
         <!-- Joint: base_link & front motor -->
-        <joint name="${prefix}_joint_front_motor" type="continuous">
-            <parent link="${prefix}_base_link"/>
-            <child link="${prefix}_front_motor_link"/>
+        <joint name="joint_front_motor" type="continuous">
+            <parent link="base_link"/>
+            <child link="front_motor_link"/>
             <origin xyz="${wheel_offset_x} ${wheel_offset_y} ${motor_wheel_offset_z}" rpy="0 0 0" />
             <axis xyz="0 0 1" rpy="0 0 0" />
@@ -233,10 +233,10 @@
         </joint>
         <!-- Transmission: front motor -->
-        <transmission name="${prefix}_joint_fmw_trans">
-            <type>transmission_interface/SimpleTransmission</type>
-            <joint name="${prefix}_joint_front_motor">
-                <hardwareInterface>hardware_interface/EffortJointInterface</hardwareInterface>
-            </joint>
-            <actuator name="${prefix}_joint_fmw_motor">
+        <transmission name="joint_fmw_trans">
+            <type>transmission_interface/SimpleTransmission</type>
+            <joint name="joint_front_motor">
+                <hardwareInterface>hardware_interface/EffortJointInterface</hardwareInterface>
+            </joint>
+            <actuator name="joint_fmw_motor">
                 <hardwareInterface>hardware_interface/EffortJointInterface</hardwareInterface>
                 <mechanicalReduction>${motor_wheel_mechanical_reduction}</mechanicalReduction>
@@ -244,5 +244,5 @@
         </transmission>
         <!-- Link: front wheel link -->
-        <link name="${prefix}_front_wheel_link">
+        <link name="front_wheel_link">
             <xacro:Wheel_Inertia    m="${wheel_mass}"
                                     ixx="${wheel_ixx}"
@@ -266,7 +266,7 @@
         </link>
         <!-- Joint: front motor & front wheel link -->
-        <joint name="${prefix}_joint_front_wheel" type="continuous">
-            <parent link="${prefix}_front_motor_link"/>
-            <child link="${prefix}_front_wheel_link"/>
+        <joint name="joint_front_wheel" type="continuous">
+            <parent link="front_motor_link"/>
+            <child link="front_wheel_link"/>
             <origin xyz="0 0 0" rpy="0 0 0" />
             <axis xyz="0 1 0" rpy="0 0 0" />
@@ -275,10 +275,10 @@
         </joint>
         <!-- Transmission: back wheel -->
-        <transmission name="${prefix}_joint_fw_trans">
-            <type>transmission_interface/SimpleTransmission</type>
-            <joint name="${prefix}_joint_front_wheel">
+        <transmission name="joint_fw_trans">
+            <type>transmission_interface/SimpleTransmission</type>
+            <joint name="joint_front_wheel">
                 <hardwareInterface>hardware_interface/VelocityJointInterface</hardwareInterface>
             </joint>
-            <actuator name="${prefix}_joint_fw_motor">
+            <actuator name="joint_fw_motor">
                 <hardwareInterface>hardware_interface/VelocityJointInterface</hardwareInterface>
                 <mechanicalReduction>${wheel_mechanical_reduction}</mechanicalReduction>
@@ -286,5 +286,5 @@
         </transmission>
         <!-- Link: left wheel link -->
-        <link name="${prefix}_left_wheel_link">
+        <link name="left_wheel_link">
             <xacro:Wheel_Inertia    m="${side_wheel_mass}"
                                     ixx="${side_wheel_ixx}"
@@ -308,7 +308,7 @@
         </link>
         <!-- Joint: base link & left wheel link -->
-        <joint name="${prefix}_joint_left_wheel" type="continuous">
-            <parent link="${prefix}_base_link"/>
-            <child link="${prefix}_left_wheel_link"/>
+        <joint name="joint_left_wheel" type="continuous">
+            <parent link="base_link"/>
+            <child link="left_wheel_link"/>
             <origin xyz="0 ${side_wheel_offset_y} ${side_wheel_offset_z}" rpy="0 0 0" />
             <axis xyz="0 1 0" rpy="0 0 0" />
@@ -317,10 +317,10 @@
         </joint>
         <!-- Transmission: left wheel -->
-        <transmission name="${prefix}_joint_lw_trans">
-            <type>transmission_interface/SimpleTransmission</type>
-            <joint name="${prefix}_joint_left_wheel">
-                <hardwareInterface>hardware_interface/EffortJointInterface</hardwareInterface>
-            </joint>
-            <actuator name="${prefix}_joint_lw_motor">
+        <transmission name="joint_lw_trans">
+            <type>transmission_interface/SimpleTransmission</type>
+            <joint name="joint_left_wheel">
+                <hardwareInterface>hardware_interface/EffortJointInterface</hardwareInterface>
+            </joint>
+            <actuator name="joint_lw_motor">
                 <hardwareInterface>hardware_interface/EffortJointInterface</hardwareInterface>
                 <mechanicalReduction>${wheel_mechanical_reduction}</mechanicalReduction>
@@ -328,5 +328,5 @@
         </transmission>
         <!-- Link: right wheel link -->
-        <link name="${prefix}_right_wheel_link">
+        <link name="right_wheel_link">
             <xacro:Wheel_Inertia    m="${side_wheel_mass}"
                                     ixx="${side_wheel_ixx}"
@@ -350,7 +350,7 @@
         </link>
         <!-- Joint: base link & right wheel link -->
-        <joint name="${prefix}_joint_right_wheel" type="continuous">
-            <parent link="${prefix}_base_link"/>
-            <child link="${prefix}_right_wheel_link"/>
+        <joint name="joint_right_wheel" type="continuous">
+            <parent link="base_link"/>
+            <child link="right_wheel_link"/>
             <origin xyz="0 -${side_wheel_offset_y} ${side_wheel_offset_z}" rpy="0 0 0" />
             <axis xyz="0 1 0" rpy="0 0 0" />
@@ -359,10 +359,10 @@
         </joint>
         <!-- Transmission: right wheel -->
-        <transmission name="${prefix}_joint_rw_trans">
-            <type>transmission_interface/SimpleTransmission</type>
-            <joint name="${prefix}_joint_right_wheel">
-                <hardwareInterface>hardware_interface/EffortJointInterface</hardwareInterface>
-            </joint>
-            <actuator name="${prefix}_joint_rw_motor">
+        <transmission name="joint_rw_trans">
+            <type>transmission_interface/SimpleTransmission</type>
+            <joint name="joint_right_wheel">
+                <hardwareInterface>hardware_interface/EffortJointInterface</hardwareInterface>
+            </joint>
+            <actuator name="joint_rw_motor">
                 <hardwareInterface>hardware_interface/EffortJointInterface</hardwareInterface>
                 <mechanicalReduction>${wheel_mechanical_reduction}</mechanicalReduction>
@@ -370,5 +370,5 @@
         </transmission>
     </xacro:macro>
-    <!-- Create DSR Body With Prefix Name -->
-    <xacro:DSR_BODY prefix="DSR"/>
+    <!-- Create DSR Body -->
+    <xacro:DSR_BODY/>
 </robot>

File: dsr_description/urdf/sensor/imu.urdf.xacro (robot description, xacro)
@@ -2,6 +2,6 @@
 <robot name="$(arg robotName)"  xmlns:xacro="http://ros.org/wiki/xacro">
     <!-- IMU SENSOR -->
-    <xacro:macro name="imu" params ="prefix x y z">
-        <link name="${prefix}_imu_link">
+    <xacro:macro name="imu" params ="x y z">
+        <link name="imu_link">
             <inertial>
                 <mass value="0.001"/>
@@ -22,9 +22,9 @@
             </collision>
         </link>
-        <joint name="${prefix}_imu_joint" type="fixed">
+        <joint name="imu_joint" type="fixed">
             <axis xyz="1 0 0"/> <!-- 0 1 0 -->
             <origin xyz="${x} ${y} ${z}"/>
-            <parent link="${prefix}_base_link"/>
-            <child link="${prefix}_imu_link"/>
+            <parent link="base_link"/>
+            <child link="imu_link"/>
         </joint>
         <gazebo>
@@ -32,5 +32,5 @@
                 <robotNamespace>$(arg robotName)</robotNamespace>
                 <topicName>imu_data</topicName>
-                <bodyName>${prefix}_imu_link</bodyName>
+                <bodyName>imu_link</bodyName>
                 <serviceName>/imu_service</serviceName>
                 <gaussianNoise>0.005</gaussianNoise>
@@ -38,4 +38,4 @@
         </gazebo>
     </xacro:macro>
-    <xacro:imu prefix="DSR" x="0" y="0" z="0.2825"/>
+    <xacro:imu x="0" y="0" z="0.2825"/>
 </robot>

File: dsr_description/urdf/sensor/lidar.urdf.xacro (robot description, xacro)
@@ -2,13 +2,13 @@
 <robot name="$(arg robotName)"  xmlns:xacro="http://ros.org/wiki/xacro">
     <!-- LIDAR SENSOR -->
-    <xacro:macro name="lidar" params ="prefix suffix x y z yaw">
-        <link name="${prefix}_laser_${suffix}"/>
-        <joint name="${prefix}_joint_laser_${suffix}" type="fixed">
+    <xacro:macro name="lidar" params ="suffix x y z yaw">
+        <link name="laser_${suffix}"/>
+        <joint name="joint_laser_${suffix}" type="fixed">
             <axis xyz="0 1 0" />
             <origin xyz="${x} ${y} ${z}" rpy="0 0 ${yaw}"/>
-            <parent link="${prefix}_base_link"/>
-            <child link="${prefix}_laser_${suffix}"/>
+            <parent link="base_link"/>
+            <child link="laser_${suffix}"/>
         </joint>
-        <gazebo reference="${prefix}_laser_${suffix}">
+        <gazebo reference="laser_${suffix}">
             <sensor type="ray" name="${suffix}_sick_sensor">
                 <pose>0 0 0 0 0 0</pose>
@@ -38,10 +38,10 @@
                     <robotNamespace>$(arg robotName)</robotNamespace>
                     <topicName>${suffix}/scan</topicName>
-                    <frameName>${prefix}_laser_${suffix}</frameName>
+                    <frameName>laser_${suffix}</frameName>
                 </plugin>
             </sensor>
         </gazebo>
     </xacro:macro>
-    <xacro:lidar prefix="DSR" suffix="front" x="0.772" y="0" z="0.14" yaw="0"/>
-    <xacro:lidar prefix="DSR" suffix="rear" x="-0.772" y="0" z="0.14" yaw="3.1416"/>
+    <xacro:lidar suffix="front" x="0.772" y="0" z="0.14" yaw="0"/>
+    <xacro:lidar suffix="rear" x="-0.772" y="0" z="0.14" yaw="3.1416"/>
 </robot>

Commit message: make some changes for ros controller

File: dsr_description/urdf/DSR_body.urdf.xacro (robot description, xacro)
@@ -149,14 +149,24 @@
         </joint>
         <!-- Transmission: back motor -->
+        <!-- <transmission name="joint_bmw_trans">
+            <type>transmission_interface/SimpleTransmission</type>
+            <joint name="joint_back_motor">
+                <hardwareInterface>hardware_interface/EffortJointInterface</hardwareInterface>
+            </joint>
+            <actuator name="joint_bmw_motor">
+                <hardwareInterface>hardware_interface/EffortJointInterface</hardwareInterface>
+                <mechanicalReduction>${motor_wheel_mechanical_reduction}</mechanicalReduction>
+            </actuator>
+        </transmission> -->
         <transmission name="joint_bmw_trans">
-            <type>transmission_interface/SimpleTransmission</type>
-            <joint name="joint_back_motor">
-                <hardwareInterface>hardware_interface/EffortJointInterface</hardwareInterface>
-            </joint>
-            <actuator name="joint_bmw_motor">
-                <hardwareInterface>hardware_interface/EffortJointInterface</hardwareInterface>
-                <mechanicalReduction>${motor_wheel_mechanical_reduction}</mechanicalReduction>
-            </actuator>
-        </transmission>
+			<type>transmission_interface/SimpleTransmission</type>
+			<joint name="joint_back_motor">
+				<hardwareInterface>hardware_interface/PositionJointInterface</hardwareInterface>
+			</joint>
+			<actuator name="joint_bmw_motor">
+                <hardwareInterface>hardware_interface/PositionJointInterface</hardwareInterface>
+				<mechanicalReduction>${motor_wheel_mechanical_reduction}</mechanicalReduction>
+			</actuator>
+		</transmission>
         <!-- Link: back wheel link -->
         <link name="back_wheel_link">
@@ -233,14 +243,24 @@
         </joint>
         <!-- Transmission: front motor -->
+        <!-- <transmission name="joint_fmw_trans">
+            <type>transmission_interface/SimpleTransmission</type>
+            <joint name="joint_front_motor">
+                <hardwareInterface>hardware_interface/EffortJointInterface</hardwareInterface>
+            </joint>
+            <actuator name="joint_fmw_motor">
+                <hardwareInterface>hardware_interface/EffortJointInterface</hardwareInterface>
+                <mechanicalReduction>${motor_wheel_mechanical_reduction}</mechanicalReduction>
+            </actuator>
+        </transmission> -->
         <transmission name="joint_fmw_trans">
-            <type>transmission_interface/SimpleTransmission</type>
-            <joint name="joint_front_motor">
-                <hardwareInterface>hardware_interface/EffortJointInterface</hardwareInterface>
-            </joint>
-            <actuator name="joint_fmw_motor">
-                <hardwareInterface>hardware_interface/EffortJointInterface</hardwareInterface>
-                <mechanicalReduction>${motor_wheel_mechanical_reduction}</mechanicalReduction>
-            </actuator>
-        </transmission>
+			<type>transmission_interface/SimpleTransmission</type>
+			<joint name="joint_front_motor">
+				<hardwareInterface>hardware_interface/PositionJointInterface</hardwareInterface>
+			</joint>
+			<actuator name="joint_fmw_motor">
+                <hardwareInterface>hardware_interface/PositionJointInterface</hardwareInterface>
+				<mechanicalReduction>${motor_wheel_mechanical_reduction}</mechanicalReduction>
+			</actuator>
+		</transmission>
         <!-- Link: front wheel link -->
         <link name="front_wheel_link">
